File: board/board.kicad_pcb (KiCad board)
At the start: 2 copper layers, 21 x 13 mm, 1 part

Commit message: initial
Parts:
- added J1: 019_100BASE-T_with_CT, on_edge:on_edge_2x05_device, F.Cu at (140.0, 96.5)
- added J2: 009_1000BASE-T, on_edge:on_edge_2x05_host, F.Cu at (161.0, 96.5)
- added J3: 004_BASE-T_CT, on_edge:on_edge_2x05_host, F.Cu at (161.0, 112.5)
- added TR1: 749013011A, b099:749013011A, F.Cu at (150.5, 97.0)
- moved LOGO1 17.7 mm to (143.5, 115.5)
Routing:
- net /eth_magnetics/CT1: track 0.00 -> 20.1 mm, vias 0 -> 2
- net /eth_magnetics/CT2: track 0.00 -> 18.5 mm
- net /eth_magnetics/RCT: track 0.00 -> 6.43 mm, vias 0 -> 1
- net /eth_magnetics/TXD+: track 0.00 -> 4.56 mm
- net /eth_magnetics/TX+: track 0.00 -> 4.56 mm
- net /eth_magnetics/TXD-: track 0.00 -> 4.33 mm
- net /eth_magnetics/TX-: track 0.00 -> 4.33 mm
- net /eth_magnetics/TCT: track 0.00 -> 4.28 mm, vias 0 -> 1
- net /eth_magnetics/RXD-: track 0.00 -> 4.14 mm
- net /eth_magnetics/RX-: track 0.00 -> 4.14 mm
- net /eth_magnetics/RXD+: track 0.00 -> 4.00 mm
- net /eth_magnetics/RX+: track 0.00 -> 4.00 mm
Other:
- board size 21 x 13 mm -> 21 x 29 mm
- board text added: "osf.004"
- board text added: "osf.009"
- board text added: "osf.019"
- board text added: "osf.b099.v0.1"
